File: Ground-Powering-Unit.kicad_sch (KiCad schematic)
At the start: 13 parts, among them J2 Conn_01x02_Pin, J3 Conn_01x02_Pin, J4 Conn_01x02_Pin, U2 LF90_TO220

Commit message: updated text in schematic
Other:
- note added: "Ground Power Unit:"
- note removed: "Remote Arming System:"
Changed lines of the file:
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@@
 		)
 	)
-	(text "Remote Arming System:"
+	(text "Ground Power Unit:"
 		(exclude_from_sim no)
 		(at 64.262 21.336 0)
@@
 		)
 		(instances
-			(project "Remote_Arming"
+			(project "Ground-Powering-Unit"
 				(path "/63b2c836-08da-46d0-ba2b-3d7f0128728d"
 					(reference "#PWR04")
@@
 		)
 		(instances
-			(project "Remote_Arming"
+			(project "Ground-Powering-Unit"
 				(path "/63b2c836-08da-46d0-ba2b-3d7f0128728d"
 					(reference "D3")
@@
 		)
 		(instances
-			(project "Remote_Arming"
+			(project "Ground-Powering-Unit"
 				(path "/63b2c836-08da-46d0-ba2b-3d7f0128728d"
 					(reference "C4")
@@
 		)
 		(instances
-			(project "Remote_Arming"
+			(project "Ground-Powering-Unit"
 				(path "/63b2c836-08da-46d0-ba2b-3d7f0128728d"
 					(reference "J2")
@@
 		)
 		(instances
-			(project "Remote_Arming"
+			(project "Ground-Powering-Unit"
 				(path "/63b2c836-08da-46d0-ba2b-3d7f0128728d"
 					(reference "#PWR07")
@@
 		)
 		(instances
-			(project "Remote_Arming"
+			(project "Ground-Powering-Unit"
 				(path "/63b2c836-08da-46d0-ba2b-3d7f0128728d"
 					(reference "#PWR010")
@@
 		)
 		(instances
-			(project "Remote_Arming"
+			(project "Ground-Powering-Unit"
 				(path "/63b2c836-08da-46d0-ba2b-3d7f0128728d"
 					(reference "L1")
@@
 		)
 		(instances
-			(project "Remote_Arming"
+			(project "Ground-Powering-Unit"
 				(path "/63b2c836-08da-46d0-ba2b-3d7f0128728d"
 					(reference "D2")
@@
 		)
 		(instances
-			(project "Remote_Arming"
+			(project "Ground-Powering-Unit"
 				(path "/63b2c836-08da-46d0-ba2b-3d7f0128728d"
 					(reference "C5")
@@
 		)
 		(instances
-			(project "Remote_Arming"
+			(project "Ground-Powering-Unit"
 				(path "/63b2c836-08da-46d0-ba2b-3d7f0128728d"
 					(reference "U2")
@@
 		)
 		(instances
-			(project "Remote_Arming"
+			(project "Ground-Powering-Unit"
 				(path "/63b2c836-08da-46d0-ba2b-3d7f0128728d"
 					(reference "#PWR03")
@@
 		)
 		(instances
-			(project "Remote_Arming"
+			(project "Ground-Powering-Unit"
 				(path "/63b2c836-08da-46d0-ba2b-3d7f0128728d"
 					(reference "C2")
@@
 		)
 		(instances
-			(project "Remote_Arming"
+			(project "Ground-Powering-Unit"
 				(path "/63b2c836-08da-46d0-ba2b-3d7f0128728d"
 					(reference "#PWR011")
@@
 		)
 		(instances
-			(project "Remote_Arming"
+			(project "Ground-Powering-Unit"
 				(path "/63b2c836-08da-46d0-ba2b-3d7f0128728d"
 					(reference "#PWR09")
@@
 		)
 		(instances
-			(project "Remote_Arming"
+			(project "Ground-Powering-Unit"
 				(path "/63b2c836-08da-46d0-ba2b-3d7f0128728d"
 					(reference "C3")
@@
 		)
 		(instances
-			(project "Remote_Arming"
+			(project "Ground-Powering-Unit"
 				(path "/63b2c836-08da-46d0-ba2b-3d7f0128728d"
 					(reference "C1")
@@
 		)
 		(instances
-			(project "Remote_Arming"
+			(project "Ground-Powering-Unit"
 				(path "/63b2c836-08da-46d0-ba2b-3d7f0128728d"
 					(reference "#PWR05")
@@
 		)
 		(instances
-			(project "Remote_Arming"
+			(project "Ground-Powering-Unit"
 				(path "/63b2c836-08da-46d0-ba2b-3d7f0128728d"
 					(reference "J4")
@@
 		)
 		(instances
-			(project "Remote_Arming"
+			(project "Ground-Powering-Unit"
 				(path "/63b2c836-08da-46d0-ba2b-3d7f0128728d"
 					(reference "#PWR06")
@@
 		)
 		(instances
-			(project "Remote_Arming"
+			(project "Ground-Powering-Unit"
 				(path "/63b2c836-08da-46d0-ba2b-3d7f0128728d"
 					(reference "#PWR08")
@@
 		)
 		(instances
-			(project "Remote_Arming"
+			(project "Ground-Powering-Unit"
 				(path "/63b2c836-08da-46d0-ba2b-3d7f0128728d"
 					(reference "J3")
@@
 		)
 		(instances
-			(project "Remote_Arming"
+			(project "Ground-Powering-Unit"
 				(path "/63b2c836-08da-46d0-ba2b-3d7f0128728d"
 					(reference "BT1")
